File: Vectrex Pad miniNeoGeo.kicad_sch (KiCad schematic)
At the start: 30 parts, among them J1 DB9_Female, SW1 SW_Push, SW2 SW_Push, SW3 SW_Push, SW4 SW_Push, SW5 SW_DP3T, SW6 SW_DP3T, U1 NE555D, U2 74LVC2G00, U3 74LVC2G32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

Commit message: Invert NAND et OR gate
It makes more sense for auto-auto-fire to be in the extreme position. To avoid generating an unwanted press while moving the switch.
Parts:
- U2: value 74LVC2G00 -> 74LVC2G32; symbol 74xGxx:74LVC2G00 -> 74xGxx:74LVC2G32
- U3: value 74LVC2G32 -> 74LVC2G00; symbol 74xGxx:74LVC2G32 -> 74xGxx:74LVC2G00
Changed lines of the file:
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@@
     (pin "2")
   )
-  (symbol (lib_id "74xGxx:74LVC2G00") (at 152.4 48.26 0) (mirror y) (unit 1)
+  (symbol (lib_name "74LVC2G32_1") (lib_id "74xGxx:74LVC2G32") (at 152.4 48.26 0) (mirror y) (unit 1)
     (in_bom yes) (on_board yes)
     (property "Reference" "U2" (id 0) (at 152.4 39.37 0))
-    (property "Value" "74LVC2G00" (id 1) (at 152.4 41.91 0))
+    (property "Value" "74LVC2G32" (id 1) (at 152.4 41.91 0))
     (property "Footprint" "Vectrex Pad miniNeoGeo:SSOP-8_2.95x2.8mm_P0.65mm" (id 2) (at 152.4 48.26 0)
       (effects (font (size 1.27 1.27)) hide)
@@
     (pin "1")
   )
-  (symbol (lib_id "74xGxx:74LVC2G32") (at 152.4 63.5 0) (mirror y) (unit 1)
+  (symbol (lib_id "74xGxx:74LVC2G00") (at 152.4 63.5 0) (mirror y) (unit 1)
     (in_bom yes) (on_board yes)
     (property "Reference" "U3" (id 0) (at 152.4 54.61 0))
-    (property "Value" "74LVC2G32" (id 1) (at 152.4 57.15 0))
+    (property "Value" "74LVC2G00" (id 1) (at 152.4 57.15 0))
     (property "Footprint" "Vectrex Pad miniNeoGeo:SSOP-8_2.95x2.8mm_P0.65mm" (id 2) (at 152.4 63.5 0)
       (effects (font (size 1.27 1.27)) hide)
@@
     (pin "1")
   )
-  (symbol (lib_id "74xGxx:74LVC2G32") (at 152.4 93.98 0) (mirror y) (unit 2)
+  (symbol (lib_id "74xGxx:74LVC2G00") (at 152.4 93.98 0) (mirror y) (unit 2)
     (in_bom yes) (on_board yes)
     (property "Reference" "U3" (id 0) (at 152.4 87.63 0))
-    (property "Value" "74LVC2G32" (id 1) (at 152.4 90.17 0))
+    (property "Value" "74LVC2G00" (id 1) (at 152.4 90.17 0))
     (property "Footprint" "Vectrex Pad miniNeoGeo:SSOP-8_2.95x2.8mm_P0.65mm" (id 2) (at 152.4 93.98 0)
       (effects (font (size 1.27 1.27)) hide)
@@
     (pin "2")
   )
-  (symbol (lib_id "74xGxx:74LVC2G00") (at 152.4 78.74 0) (mirror y) (unit 2)
+  (symbol (lib_name "74LVC2G32_2") (lib_id "74xGxx:74LVC2G32") (at 152.4 78.74 0) (mirror y) (unit 2)
     (in_bom yes) (on_board yes)
     (property "Reference" "U2" (id 0) (at 152.4 72.39 0))
-    (property "Value" "74LVC2G00" (id 1) (at 152.4 74.93 0))
+    (property "Value" "74LVC2G32" (id 1) (at 152.4 74.93 0))
     (property "Footprint" "Vectrex Pad miniNeoGeo:SSOP-8_2.95x2.8mm_P0.65mm" (id 2) (at 152.4 78.74 0)
       (effects (font (size 1.27 1.27)) hide)
@@
     )
     (path "/02d454b8-c745-4892-9416-6585879612b9"
-      (reference "U2") (unit 1) (value "74LVC2G00") (footprint "Vectrex Pad miniNeoGeo:SSOP-8_2.95x2.8mm_P0.65mm")
+      (reference "U2") (unit 1) (value "74LVC2G32") (footprint "Vectrex Pad miniNeoGeo:SSOP-8_2.95x2.8mm_P0.65mm")
     )
     (path "/bdb16a67-44da-4c3e-afd7-840af86d0645"
-      (reference "U2") (unit 2) (value "74LVC2G00") (footprint "Vectrex Pad miniNeoGeo:SSOP-8_2.95x2.8mm_P0.65mm")
+      (reference "U2") (unit 2) (value "74LVC2G32") (footprint "Vectrex Pad miniNeoGeo:SSOP-8_2.95x2.8mm_P0.65mm")
     )
     (path "/97ed9c90-1981-4a69-9e3d-c5b9aacd2ee6"
-      (reference "U3") (unit 1) (value "74LVC2G32") (footprint "Vectrex Pad miniNeoGeo:SSOP-8_2.95x2.8mm_P0.65mm")
+      (reference "U3") (unit 1) (value "74LVC2G00") (footprint "Vectrex Pad miniNeoGeo:SSOP-8_2.95x2.8mm_P0.65mm")
     )
     (path "/a0fa3fdb-8123-4bdc-b653-2a451c8f37f3"
-      (reference "U3") (unit 2) (value "74LVC2G32") (footprint "Vectrex Pad miniNeoGeo:SSOP-8_2.95x2.8mm_P0.65mm")
+      (reference "U3") (unit 2) (value "74LVC2G00") (footprint "Vectrex Pad miniNeoGeo:SSOP-8_2.95x2.8mm_P0.65mm")
     )
     (path "/cde73a30-8337-49f6-b83b-7f969bf135ef"
